File: pcb/splitflap.kicad_pcb (KiCad board)
At the start: 2 copper layers, 160 x 100 mm, 19 parts, among them J1 Conn_01x01, J2 Conn_01x01, J3 Screw_Terminal_01x02, T1 Transformer_1P_2S, T2 Transformer_1P_1S, U1 LD1117S33TR_SOT223

Commit message: 100x100-platine
Parts:
- moved REF** 195.0 mm to (-111.8, -14.0)
Routing:
- net +3V3: track 207.8 -> 0.00 mm
- net 48VAC_N: track 193.8 -> 0.00 mm
- net 48VAC_L: track 140.7 -> 0.00 mm
- net /SENSOR_IN: track 102.8 -> 0.00 mm
- net 230VAC_N: track 89.1 -> 0.00 mm
- net /MOTOR: track 63.2 -> 0.00 mm
- net /SENSOR1: track 58.6 -> 0.00 mm
- net /SENSOR2: track 57.9 -> 0.00 mm
- net Net-(C1-Pad1): track 55.0 -> 0.00 mm
- net 230VAC_L: track 48.5 -> 0.00 mm
- net Net-(D1-Pad4): track 25.2 -> 0.00 mm
- net Net-(BKOUT_L1-Pad1): track 19.4 -> 0.00 mm
- net Net-(BKOUT_R1-Pad1): track 19.1 -> 0.00 mm
- net Net-(D1-Pad2): track 18.1 -> 0.00 mm
- net Net-(BKOUT_R1-Pad9): track 10.2 -> 0.00 mm
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Other:
- outline, holes or cut-outs redrawn

Commit message: footprints
Parts:
- removed C_DATA1, C_POWER1: DB9_Female, Connectors_DSub:DSUB-9_Female_Horizontal_Pitch2.77x2.54mm_EdgePinOffset9.40mm
- removed J1, J2: Conn_01x01, Wire_Pads:SolderWirePad_single_1-2mmDrill
- removed the REF** at (-111.8, -14.0)
- removed T1: Transformer_1P_2S, special:Transformer_CHK_EI48-10VA_2xSec_BLOCK
- removed T2: Transformer_1P_1S, Transformers_THT:Transformer_CHK_EI30-2VA_1xSec
- added DATA_CONNECTOR1: DB25_Female, special:DSUB-25_Female_Horizontal_Pitch2.77x2.54mm_EdgePinOffset9.40mm_CLICK, F.Cu at (182.9, 86.1)
- added POWER_CONNECTOR1: DB9_Female, special:DSUB-9_Female_Horizontal_Pitch2.77x2.54mm_EdgePinOffset9.40mm_CLICK, F.Cu at (106.7, 73.8)
- added REF**: MountingHole_3.2mm_M3, Mounting_Holes:MountingHole_3.2mm_M3, F.Cu at (99.8, 135.8)
- added REF**: MountingHole_3.2mm_M3, Mounting_Holes:MountingHole_3.2mm_M3, F.Cu at (99.8, 45.8)
- added REF**: MountingHole_3.2mm_M3, Mounting_Holes:MountingHole_3.2mm_M3, F.Cu at (189.8, 45.8)
- added REF**: MountingHole_3.2mm_M3, Mounting_Holes:MountingHole_3.2mm_M3, F.Cu at (189.8, 135.8)
- added RV1: Varistor, Varistors:RV_Disc_D12_W3.9_P7.5, F.Cu at (106.8, 91.8)
- added TRAFO1: Transformer_1P_2S, special:Transformer_CHK_EI48-10VA_2xSec_BLOCK, F.Cu at (143.8, 55.8)
- added TRAFO2: Transformer_1P_1S, special:Transformer_CHK_EI30-2VA_1xSec, F.Cu at (158.8, 46.8)
- J3: footprint TerminalBlocks_Phoenix:TerminalBlock_Phoenix_PT-3.5mm_2pol -> TerminalBlock_MetzConnect:TerminalBlock_MetzConnect_Type171_RT13702HBWC_Pitch7.50mm
- moved GND_BREAK1 91.6 mm to (111.8, 135.8), turned to 180 degrees
- moved VCC_BREAK1 88.5 mm to (107.2, 133.2), turned to 0 degrees
- moved BKOUT_R1 74.0 mm to (166.4, 136.6), turned to 270 degrees
- moved ESP32_R1 68.0 mm to (166.4, 131.5), turned to 270 degrees
- moved D1 62.0 mm to (153.8, 73.8)
- moved C3 52.3 mm to (170.8, 74.8), turned to 0 degrees
- moved BKOUT_L1 51.1 mm to (166.4, 103.6), turned to 270 degrees
- moved U1 50.3 mm to (174.8, 80.8), turned to 180 degrees
- moved ESP32_L1 50.0 mm to (166.4, 108.7), turned to 270 degrees
- moved J3 49.2 mm to (101.8, 98.8), turned to 270 degrees
- moved C1 45.6 mm to (157.8, 86.8)
- moved C2 43.1 mm to (171.0, 86.1), turned to 0 degrees
Connections:
- net /MOTOR renamed /MOTOR1
- net /SENSOR1 renamed /FSENSOR1
- net /SENSOR2 renamed /HSENSOR1
- net /SENSOR_IN renamed /SENSOR_IN_1
- net Net-(BKOUT_L1-Pad1) renamed /+3.3V_ESP
- net Net-(BKOUT_L1-Pad10) renamed /HSENSOR5
- net Net-(BKOUT_L1-Pad11) renamed /FSENSOR6
- net Net-(BKOUT_L1-Pad12) renamed /HSENSOR6
- net Net-(BKOUT_L1-Pad4) renamed /SENSOR_IN_2
- net Net-(BKOUT_L1-Pad5) renamed /SENSOR_IN_3
- net Net-(BKOUT_L1-Pad6) renamed /SENSOR_IN_4
- net Net-(BKOUT_L1-Pad7) renamed /SENSOR_IN_5
- net Net-(BKOUT_L1-Pad8) renamed /SENSOR_IN_6
- net Net-(BKOUT_L1-Pad9) renamed /FSENSOR5
- net Net-(BKOUT_R1-Pad10) renamed /HSENSOR2
- net Net-(BKOUT_R1-Pad11) renamed /FSENSOR3
- net Net-(BKOUT_R1-Pad12) renamed /HSENSOR3
- net Net-(BKOUT_R1-Pad13) renamed /FSENSOR4
- net Net-(BKOUT_R1-Pad14) renamed /HSENSOR4
- net Net-(BKOUT_R1-Pad15) renamed /MOTOR2
- net Net-(BKOUT_R1-Pad16) renamed /MOTOR3
- net Net-(BKOUT_R1-Pad17) renamed /MOTOR4
- net Net-(BKOUT_R1-Pad18) renamed /MOTOR5
- net Net-(BKOUT_R1-Pad19) renamed /MOTOR6
- net Net-(BKOUT_R1-Pad9) renamed /FSENSOR2
- BKOUT_L1 pad 14: Net-(BKOUT_L1-Pad14) -> /GND_ESP
- BKOUT_R1 pad 1: Net-(BKOUT_R1-Pad1) -> /GND_ESP
- BKOUT_R1 pad 7: Net-(BKOUT_R1-Pad7) -> /GND_ESP
- ESP32_L1 pad 14: Net-(BKOUT_L1-Pad14) -> /GND_ESP
- ESP32_R1 pad 1: Net-(BKOUT_R1-Pad1) -> /GND_ESP
- ESP32_R1 pad 7: Net-(BKOUT_R1-Pad7) -> /GND_ESP
- GND_BREAK1 pad 2: Net-(BKOUT_R1-Pad1) -> /GND_ESP
Routing:
- net 230VAC_L: track 0.00 -> 121.8 mm
- net 230VAC_N: track 0.00 -> 96.4 mm
- net /+3.3V_ESP: track 0.00 -> 79.0 mm, vias 0 -> 2
- net 48VAC_N: track 0.00 -> 32.5 mm
- net Net-(D1-Pad4): track 0.00 -> 17.9 mm
- net Net-(D1-Pad2): track 0.00 -> 16.8 mm
- net Net-(TRAFO1-Pad11): track 0.00 -> 15.5 mm
- net 48VAC_L: track 0.00 -> 14.5 mm
- removed copper zone on B.Cu, net GND
Other:
- board size 160 x 100 mm -> 100 x 100 mm

Commit message: wiring
Parts:
- DATA_CONNECTOR1: footprint special:DSUB-25_Female_Horizontal_Pitch2.77x2.54mm_EdgePinOffset9.40mm_CLICK -> DSUB-25_Female_Horizontal_Pitch2.77x2.54mm_EdgePinOffset9.40mm_CLICK
- POWER_CONNECTOR1: footprint special:DSUB-9_Female_Horizontal_Pitch2.77x2.54mm_EdgePinOffset9.40mm_CLICK -> DSUB-9_Female_Horizontal_Pitch2.77x2.54mm_EdgePinOffset9.40mm_CLICK
Connections:
- DATA_CONNECTOR1 pad 13: GND -> /GND_ESP
Routing:
- net GND: track 0.00 -> 161.1 mm, vias 0 -> 4
- net /FSENSOR2: track 0.00 -> 155.1 mm
- net /HSENSOR2: track 0.00 -> 153.5 mm, vias 0 -> 2
- net +3V3: track 0.00 -> 153.0 mm, vias 0 -> 2
- net /MOTOR2: track 0.00 -> 93.3 mm, vias 0 -> 2
- net /MOTOR3: track 0.00 -> 89.7 mm, vias 0 -> 2
- net /+3.3V_ESP: track 79.0 -> 168.7 mm, vias 2 -> 4
- net /MOTOR4: track 0.00 -> 87.3 mm, vias 0 -> 2
- net /MOTOR5: track 0.00 -> 85.5 mm, vias 0 -> 2
- net /MOTOR6: track 0.00 -> 82.5 mm, vias 0 -> 2
- net /HSENSOR4: track 0.00 -> 75.1 mm, vias 0 -> 2
- net /HSENSOR1: track 0.00 -> 73.8 mm, vias 0 -> 2
- net /FSENSOR4: track 0.00 -> 71.5 mm, vias 0 -> 2
- net /HSENSOR3: track 0.00 -> 68.3 mm, vias 0 -> 2
- net /FSENSOR1: track 0.00 -> 67.0 mm, vias 0 -> 2
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- added copper zone on B.Cu, net /GND_ESP

Commit message: powerground
Parts:
- added REF**: VIA-0.6mm, special:VIA-0.6mm, F.Cu at (106.8, 119.9)
- added REF**: VIA-0.6mm, special:VIA-0.6mm, F.Cu at (114.8, 121.9)
- added REF**: VIA-0.6mm, special:VIA-0.6mm, F.Cu at (106.8, 123.9)
- added REF**: VIA-0.6mm, special:VIA-0.6mm, F.Cu at (108.8, 123.9)
- added REF**: VIA-0.6mm, special:VIA-0.6mm, F.Cu at (110.8, 123.9)
- added REF**: VIA-0.6mm, special:VIA-0.6mm, F.Cu at (112.8, 123.9)
- added REF**: VIA-0.6mm, special:VIA-0.6mm, F.Cu at (114.8, 123.9)
- added REF**: VIA-0.6mm, special:VIA-0.6mm, F.Cu at (106.8, 125.9)
- added REF**: VIA-0.6mm, special:VIA-0.6mm, F.Cu at (108.8, 125.9)
- added REF**: VIA-0.6mm, special:VIA-0.6mm, F.Cu at (110.8, 125.9)
- added REF**: VIA-0.6mm, special:VIA-0.6mm, F.Cu at (112.8, 125.9)
- added REF**: VIA-0.6mm, special:VIA-0.6mm, F.Cu at (108.8, 119.9)
- added REF**: VIA-0.6mm, special:VIA-0.6mm, F.Cu at (114.8, 125.9)
- added REF**: VIA-0.6mm, special:VIA-0.6mm, F.Cu at (106.8, 127.9)
- added REF**: VIA-0.6mm, special:VIA-0.6mm, F.Cu at (108.8, 127.9)
- added REF**: VIA-0.6mm, special:VIA-0.6mm, F.Cu at (110.8, 127.9)
- added REF**: VIA-0.6mm, special:VIA-0.6mm, F.Cu at (112.8, 127.9)
- added REF**: VIA-0.6mm, special:VIA-0.6mm, F.Cu at (114.8, 127.9)
- added REF**: VIA-0.6mm, special:VIA-0.6mm, F.Cu at (150.8, 99.8)
- added REF**: VIA-0.6mm, special:VIA-0.6mm, F.Cu at (148.8, 99.8)
- added REF**: VIA-0.6mm, special:VIA-0.6mm, F.Cu at (146.8, 99.8)
- added REF**: VIA-0.6mm, special:VIA-0.6mm, F.Cu at (144.8, 99.8)
- added REF**: VIA-0.6mm, special:VIA-0.6mm, F.Cu at (110.8, 119.9)
- added REF**: VIA-0.6mm, special:VIA-0.6mm, F.Cu at (142.8, 99.8)
- added REF**: VIA-0.6mm, special:VIA-0.6mm, F.Cu at (140.8, 99.8)
- added REF**: VIA-0.6mm, special:VIA-0.6mm, F.Cu at (138.8, 99.8)
- added REF**: VIA-0.6mm, special:VIA-0.6mm, F.Cu at (136.8, 99.8)
- added REF**: VIA-0.6mm, special:VIA-0.6mm, F.Cu at (134.8, 99.8)
- added REF**: VIA-0.6mm, special:VIA-0.6mm, F.Cu at (132.8, 99.8)
- added REF**: VIA-0.6mm, special:VIA-0.6mm, F.Cu at (190.8, 69.8)
- added REF**: VIA-0.6mm, special:VIA-0.6mm, F.Cu at (188.8, 69.8)
- added REF**: VIA-0.6mm, special:VIA-0.6mm, F.Cu at (186.8, 69.8)
- added REF**: VIA-0.6mm, special:VIA-0.6mm, F.Cu at (184.8, 69.8)
- added REF**: VIA-0.6mm, special:VIA-0.6mm, F.Cu at (112.8, 119.9)
- added REF**: VIA-0.6mm, special:VIA-0.6mm, F.Cu at (182.8, 69.8)
- added REF**: VIA-0.6mm, special:VIA-0.6mm, F.Cu at (190.8, 67.8)
- added REF**: VIA-0.6mm, special:VIA-0.6mm, F.Cu at (188.8, 67.8)
- added REF**: VIA-0.6mm, special:VIA-0.6mm, F.Cu at (186.8, 67.8)
- added REF**: VIA-0.6mm, special:VIA-0.6mm, F.Cu at (184.8, 67.8)
- added REF**: VIA-0.6mm, special:VIA-0.6mm, F.Cu at (182.8, 67.8)
- added REF**: VIA-0.6mm, special:VIA-0.6mm, F.Cu at (190.8, 65.8)
- added REF**: VIA-0.6mm, special:VIA-0.6mm, F.Cu at (188.8, 65.8)
- added REF**: VIA-0.6mm, special:VIA-0.6mm, F.Cu at (186.8, 65.8)
- added REF**: VIA-0.6mm, special:VIA-0.6mm, F.Cu at (184.8, 65.8)
- added REF**: VIA-0.6mm, special:VIA-0.6mm, F.Cu at (114.8, 119.9)
- added REF**: VIA-0.6mm, special:VIA-0.6mm, F.Cu at (182.8, 65.8)
- added REF**: VIA-0.6mm, special:VIA-0.6mm, F.Cu at (190.8, 63.8)
- added REF**: VIA-0.6mm, special:VIA-0.6mm, F.Cu at (188.8, 63.8)
- added REF**: VIA-0.6mm, special:VIA-0.6mm, F.Cu at (186.8, 63.8)
- added REF**: VIA-0.6mm, special:VIA-0.6mm, F.Cu at (184.8, 63.8)
- added REF**: VIA-0.6mm, special:VIA-0.6mm, F.Cu at (182.8, 63.8)
- added REF**: VIA-0.6mm, special:VIA-0.6mm, F.Cu at (190.8, 61.8)
- added REF**: VIA-0.6mm, special:VIA-0.6mm, F.Cu at (188.8, 61.8)
- added REF**: VIA-0.6mm, special:VIA-0.6mm, F.Cu at (186.8, 61.8)
- added REF**: VIA-0.6mm, special:VIA-0.6mm, F.Cu at (184.8, 61.8)
- added REF**: VIA-0.6mm, special:VIA-0.6mm, F.Cu at (106.8, 121.9)
- added REF**: VIA-0.6mm, special:VIA-0.6mm, F.Cu at (182.8, 61.8)
- added REF**: VIA-0.6mm, special:VIA-0.6mm, F.Cu at (152.3, 129.2)
- added REF**: VIA-0.6mm, special:VIA-0.6mm, F.Cu at (152.2, 134.0)
- added REF**: VIA-0.6mm, special:VIA-0.6mm, F.Cu at (150.1, 134.0)
- added REF**: VIA-0.6mm, special:VIA-0.6mm, F.Cu at (108.8, 121.9)
- added REF**: VIA-0.6mm, special:VIA-0.6mm, F.Cu at (110.8, 121.9)
- added REF**: VIA-0.6mm, special:VIA-0.6mm, F.Cu at (112.8, 121.9)
Routing:
- net /GND_ESP: track 15.2 -> 0.00 mm
- net /SENSOR_IN_4: track 49.8 -> 48.8 mm
- added copper zone on F.Cu, net /GND_ESP
