File: pcb/splitflap.kicad_pcb (KiCad board)
At the start: 2 copper layers, 100 x 100 mm, 84 parts, among them J3 Screw_Terminal_01x02, U1 LD1117S33TR_SOT223

Commit message: labels
Other:
- board text added: "Das große Klappern"
- board text added: "Fallblatt v1.0"
Changed lines of the file:
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@@
     (links 153)
     (no_connects 0)
-    (area 84.455 39.325 205.265 145.685239)
+    (area 94.749999 40.749999 194.850001 140.850001)
     (thickness 1.6)
-    (drawings 8)
+    (drawings 10)
     (tracks 465)
     (zones 0)
@@
     (descr "25-pin D-Sub connector, horizontal/angled (90 deg), THT-mount, female, pitch 2.77x2.54mm, pin-PCB-offset 9.4mm, see http://docs-europe.electrocomponents.com/webdocs/1585/0900766b81585df2.pdf")
     (tags "25-pin D-Sub connector horizontal angled 90deg THT female pitch 2.77x2.54mm pin-PCB-offset 9.4mm")
-    (fp_text reference DATA_CONNECTOR1 (at -16.62 -1.8 90) (layer F.SilkS)
+    (fp_text reference DATA_CONNECTOR1 (at -16.68 5.92 90) (layer F.SilkS)
       (effects (font (size 1 1) (thickness 0.15)))
     )
@@
     (descr "9-pin D-Sub connector, horizontal/angled (90 deg), THT-mount, female, pitch 2.77x2.54mm, pin-PCB-offset 9.4mm, see http://docs-europe.electrocomponents.com/webdocs/1585/0900766b81585df2.pdf")
     (tags "9-pin D-Sub connector horizontal angled 90deg THT female pitch 2.77x2.54mm pin-PCB-offset 9.4mm")
-    (fp_text reference POWER_CONNECTOR1 (at -5.54 -1.8 270) (layer F.SilkS)
+    (fp_text reference POWER_CONNECTOR1 (at -5.55 9.34 270) (layer F.SilkS)
       (effects (font (size 1 1) (thickness 0.15)))
     )
@@
     (descr "C, Rect series, Radial, pin pitch=2.50mm, , length*width=4*2.5mm^2, Capacitor")
     (tags "C Rect series Radial pin pitch 2.50mm  length 4mm width 2.5mm Capacitor")
-    (fp_text reference C2 (at 1.25 -2.56) (layer F.SilkS)
+    (fp_text reference C2 (at 5.2 -0.02) (layer F.SilkS)
       (effects (font (size 1 1) (thickness 0.15)))
     )
@@
     (descr "CP, Radial series, Radial, pin pitch=2.00mm, , diameter=4mm, Electrolytic Capacitor")
     (tags "CP Radial series Radial pin pitch 2.00mm  diameter 4mm Electrolytic Capacitor")
-    (fp_text reference C3 (at 1 -3.31) (layer F.SilkS)
+    (fp_text reference C3 (at -3 0) (layer F.SilkS)
       (effects (font (size 1 1) (thickness 0.15)))
     )
@@
     (descr "4-lead round diode bridge package, diameter 8.9mm, pin pitch 5.08mm, see http://cdn-reichelt.de/documents/datenblatt/A400/W005M-W10M_SEP.PDF")
     (tags "diode bridge 8.9mm 8.85mm WOB pitch 5.08mm")
-    (fp_text reference D1 (at 2.54 -2.794) (layer F.SilkS)
+    (fp_text reference D1 (at 3.1 8.1) (layer F.SilkS)
       (effects (font (size 1 1) (thickness 0.15)))
     )
@@
     (descr "TO-220-3, Vertical, RM 2.54mm")
     (tags "TO-220-3 Vertical RM 2.54mm")
-    (fp_text reference U1 (at 2.54 -3.62 180) (layer F.SilkS)
+    (fp_text reference U1 (at 9.2 0 180) (layer F.SilkS)
       (effects (font (size 1 1) (thickness 0.15)))
     )
@@
     (descr "Through hole straight socket strip, 1x20, 2.54mm pitch, single row")
     (tags "Through hole socket strip THT 1x20 2.54mm single row")
-    (fp_text reference ESP32_R1 (at 0 -2.33 270) (layer F.SilkS)
+    (fp_text reference ESP32_R1 (at -0.01 -5.63 360) (layer F.SilkS)
       (effects (font (size 1 1) (thickness 0.15)))
     )
@@
     (descr "Through hole straight socket strip, 1x20, 2.54mm pitch, single row")
     (tags "Through hole socket strip THT 1x20 2.54mm single row")
-    (fp_text reference BKOUT_L1 (at 0 -2.33 270) (layer F.SilkS)
+    (fp_text reference BKOUT_L1 (at -2.67 45.97 360) (layer F.SilkS)
       (effects (font (size 1 1) (thickness 0.15)))
     )
@@
     (descr "Through hole straight socket strip, 1x20, 2.54mm pitch, single row")
     (tags "Through hole socket strip THT 1x20 2.54mm single row")
-    (fp_text reference BKOUT_R1 (at 0 -2.33 270) (layer F.SilkS)
+    (fp_text reference BKOUT_R1 (at -0.09 -5.73 360) (layer F.SilkS)
       (effects (font (size 1 1) (thickness 0.15)))
     )
@@
     (descr "Through hole straight socket strip, 1x20, 2.54mm pitch, single row")
     (tags "Through hole socket strip THT 1x20 2.54mm single row")
-    (fp_text reference ESP32_L1 (at 0 -2.33 270) (layer F.SilkS)
+    (fp_text reference ESP32_L1 (at 2.75 46.07 360) (layer F.SilkS)
       (effects (font (size 1 1) (thickness 0.15)))
     )
@@
     (tags "mounting hole 3.2mm no annular m3")
     (attr virtual)
-    (fp_text reference REF** (at 0 -4.2) (layer F.SilkS)
+    (fp_text reference REF** (at 0 -4.2) (layer F.SilkS) hide
       (effects (font (size 1 1) (thickness 0.15)))
     )
@@
     (tags "mounting hole 3.2mm no annular m3")
     (attr virtual)
-    (fp_text reference REF** (at 0 -4.2) (layer F.SilkS)
+    (fp_text reference REF** (at 0 -4.2) (layer F.SilkS) hide
       (effects (font (size 1 1) (thickness 0.15)))
     )
@@
     (tags "mounting hole 3.2mm no annular m3")
     (attr virtual)
-    (fp_text reference REF** (at 0 -4.2) (layer F.SilkS)
+    (fp_text reference REF** (at 0 -4.2) (layer F.SilkS) hide
       (effects (font (size 1 1) (thickness 0.15)))
     )
@@
     (tags "mounting hole 3.2mm no annular m3")
     (attr virtual)
-    (fp_text reference REF** (at 0 -4.2) (layer F.SilkS)
+    (fp_text reference REF** (at 0 -4.2) (layer F.SilkS) hide
       (effects (font (size 1 1) (thickness 0.15)))
     )
@@
       (net 51 /GND_ESP) (zone_connect 2))
   )
+  (gr_text "Das große Klappern" (at 124.3 98.8) (layer F.SilkS)
+    (effects (font (size 0.8 0.8) (thickness 0.15)))
+  )
+  (gr_text "Fallblatt v1.0" (at 124.3 96.8) (layer F.SilkS)
+    (effects (font (size 1.5 1.5) (thickness 0.3)))
+  )
   (gr_line (start 194.8 45.8) (end 194.8 135.8) (angle 90) (layer Edge.Cuts) (width 0.1))

Commit message: labels
Other:
- board text added: "6-Fach-Ansteuerungseinheit"
- board text added: "X"
Changed lines of the file:
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@@
     (area 94.749999 40.749999 194.850001 140.850001)
     (thickness 1.6)
-    (drawings 10)
+    (drawings 16)
     (tracks 465)
     (zones 0)
@@
     (descr "Through hole straight socket strip, 1x20, 2.54mm pitch, single row")
     (tags "Through hole socket strip THT 1x20 2.54mm single row")
-    (fp_text reference BKOUT_L1 (at -2.67 45.97 360) (layer F.SilkS)
+    (fp_text reference BKOUT_L1 (at -2.67 42.97 360) (layer F.SilkS)
       (effects (font (size 1 1) (thickness 0.15)))
     )
@@
     (descr "Through hole straight socket strip, 1x20, 2.54mm pitch, single row")
     (tags "Through hole socket strip THT 1x20 2.54mm single row")
-    (fp_text reference ESP32_L1 (at 2.75 46.07 360) (layer F.SilkS)
+    (fp_text reference ESP32_L1 (at 2.75 43.27 360) (layer F.SilkS)
       (effects (font (size 1 1) (thickness 0.15)))
     )
@@
       (net 51 /GND_ESP) (zone_connect 2))
   )
-  (gr_text "Das große Klappern" (at 124.3 98.8) (layer F.SilkS)
+  (gr_text X (at 118.1 139.4) (layer F.SilkS)
+    (effects (font (size 1.5 1.5) (thickness 0.3)))
+  )
+  (gr_text X (at 118.1 128.7) (layer F.SilkS)
+    (effects (font (size 1.5 1.5) (thickness 0.3)))
+  )
+  (gr_text X (at 118.1 111.5) (layer F.SilkS)
+    (effects (font (size 1.5 1.5) (thickness 0.3)))
+  )
+  (gr_text X (at 118.1 106.2) (layer F.SilkS)
+    (effects (font (size 1.5 1.5) (thickness 0.3)))
+  )
+  (gr_text X (at 118.1 100.8) (layer F.SilkS)
+    (effects (font (size 1.5 1.5) (thickness 0.3)))
+  )
+  (gr_text 6-Fach-Ansteuerungseinheit (at 144.3 96.7) (layer F.SilkS)
     (effects (font (size 0.8 0.8) (thickness 0.15)))
   )
-  (gr_text "Fallblatt v1.0" (at 124.3 96.8) (layer F.SilkS)
+  (gr_text "Das große Klappern" (at 126.4 98.3) (layer F.SilkS)
+    (effects (font (size 0.8 0.8) (thickness 0.15)))
+  )
+  (gr_text "Fallblatt v1.0" (at 126.4 96.3) (layer F.SilkS)
     (effects (font (size 1.5 1.5) (thickness 0.3)))
   )
