File: pcb/splitflap.sch (KiCad schematic (older format))
At the start: 18 parts, among them J1 Conn_01x01, J2 Conn_01x01, J3 Screw_Terminal_01x02, T1 Transformer_1P_2S, T2 Transformer_1P_1S, U1 LD1117S33TR_SOT223

Commit message: footprints
Parts:
- removed C_DATA1: DB9_Female, Connectors_DSub:DSUB-9_Female_Horizontal_Pitch2.77x2.54mm_EdgePinOffset9.40mm, symbol DB9_Female
- removed J1, J2: Conn_01x01, Wire_Pads:SolderWirePad_single_1-2mmDrill, symbol Conn_01x01
- added DATA_CONNECTOR1: DB25_Female, special:DSUB-25_Female_Horizontal_Pitch2.77x2.54mm_EdgePinOffset9.40mm_CLICK, symbol DB25_Female
- added RV1: Varistor, Varistors:RV_Disc_D12_W3.9_P7.5, symbol Varistor
- J3: footprint TerminalBlocks_Phoenix:TerminalBlock_Phoenix_PT-3.5mm_2pol -> TerminalBlock_MetzConnect:TerminalBlock_MetzConnect_Type171_RT13702HBWC_Pitch7.50mm
- POWER_CONNECTOR1: renamed from C_POWER1; footprint Connectors_DSub:DSUB-9_Female_Horizontal_Pitch2.77x2.54mm_EdgePinOffset9.40mm -> special:DSUB-9_Female_Horizontal_Pitch2.77x2.54mm_EdgePinOffset9.40mm_CLICK
- TRAFO2: renamed from T2; footprint Transformers_THT:Transformer_CHK_EI30-2VA_1xSec -> special:Transformer_CHK_EI30-2VA_1xSec
- renumbered T1 to TRAFO1
Connections:
- net +3V3: no longer POWER_CONNECTOR1.5
- net 230VAC_L: now also RV1.1
- net 230VAC_N: now also RV1.2
- net GND: now also DATA_CONNECTOR1.13; no longer POWER_CONNECTOR1.9
- net +3.3V_ESP: now reaches BKOUT_L1.1 (Pin_1), ESP32_L1.1 (Pin_1), VCC_BREAK1.2
- net +3.3V_ESP: now also POWER_CONNECTOR1.5
- net HSENSOR5: now reaches BKOUT_L1.10 (Pin_10), ESP32_L1.10 (Pin_10)
- net HSENSOR5: now also DATA_CONNECTOR1.23 (P23)
- net FSENSOR6: now reaches BKOUT_L1.11 (Pin_11), ESP32_L1.11 (Pin_11)
- net FSENSOR6: now also DATA_CONNECTOR1.12
- net HSENSOR6: now reaches BKOUT_L1.12 (Pin_12), ESP32_L1.12 (Pin_12)
- net HSENSOR6: now also DATA_CONNECTOR1.25 (P25)
- net GND_ESP: now reaches BKOUT_L1.14 (Pin_14), ESP32_L1.14 (Pin_14)
- net GND_ESP: now also BKOUT_R1.1 (Pin_1), BKOUT_R1.7 (Pin_7), ESP32_R1.1 (Pin_1), ESP32_R1.7 (Pin_7), GND_BREAK1.2, POWER_CONNECTOR1.9
- net SENSOR_IN_2: now reaches BKOUT_L1.4 (Pin_4), ESP32_L1.4 (Pin_4)
- net SENSOR_IN_2: now also DATA_CONNECTOR1.16 (P16)
- net SENSOR_IN_3: now reaches BKOUT_L1.5 (Pin_5), ESP32_L1.5 (Pin_5)
- net SENSOR_IN_3: now also DATA_CONNECTOR1.18 (P18)
- net SENSOR_IN_4: now reaches BKOUT_L1.6 (Pin_6), ESP32_L1.6 (Pin_6)
- net SENSOR_IN_4: now also DATA_CONNECTOR1.20 (P20)
- net SENSOR_IN_5: now reaches BKOUT_L1.7 (Pin_7), ESP32_L1.7 (Pin_7)
- net SENSOR_IN_5: now also DATA_CONNECTOR1.22 (P22)
- net SENSOR_IN_6: now reaches BKOUT_L1.8 (Pin_8), ESP32_L1.8 (Pin_8)
- net SENSOR_IN_6: now also DATA_CONNECTOR1.24 (P24)
- net FSENSOR5: now reaches BKOUT_L1.9 (Pin_9), ESP32_L1.9 (Pin_9)
- net FSENSOR5: now also DATA_CONNECTOR1.10
- net HSENSOR2: now reaches BKOUT_R1.10 (Pin_10), ESP32_R1.10 (Pin_10)
- net HSENSOR2: now also DATA_CONNECTOR1.17 (P17)
- net FSENSOR3: now reaches BKOUT_R1.11 (Pin_11), ESP32_R1.11 (Pin_11)
- net FSENSOR3: now also DATA_CONNECTOR1.6
- net HSENSOR3: now reaches BKOUT_R1.12 (Pin_12), ESP32_R1.12 (Pin_12)
- net HSENSOR3: now also DATA_CONNECTOR1.19 (P19)
- net FSENSOR4: now reaches BKOUT_R1.13 (Pin_13), ESP32_R1.13 (Pin_13)
- net FSENSOR4: now also DATA_CONNECTOR1.8
- net HSENSOR4: now reaches BKOUT_R1.14 (Pin_14), ESP32_R1.14 (Pin_14)
- net HSENSOR4: now also DATA_CONNECTOR1.21 (P21)
- net MOTOR2: now reaches BKOUT_R1.15 (Pin_15), ESP32_R1.15 (Pin_15)
- net MOTOR2: now also DATA_CONNECTOR1.3
- net MOTOR3: now reaches BKOUT_R1.16 (Pin_16), ESP32_R1.16 (Pin_16)
- net MOTOR3: now also DATA_CONNECTOR1.5
- net MOTOR4: now reaches BKOUT_R1.17 (Pin_17), ESP32_R1.17 (Pin_17)
- net MOTOR4: now also DATA_CONNECTOR1.7
- net MOTOR5: now reaches BKOUT_R1.18 (Pin_18), ESP32_R1.18 (Pin_18)
- net MOTOR5: now also DATA_CONNECTOR1.9
- net MOTOR6: now reaches BKOUT_R1.19 (Pin_19), ESP32_R1.19 (Pin_19)
- net MOTOR6: now also DATA_CONNECTOR1.11
- net FSENSOR2: now reaches BKOUT_R1.9 (Pin_9), ESP32_R1.9 (Pin_9)
- net FSENSOR2: now also DATA_CONNECTOR1.4
- net MOTOR renamed MOTOR1
- net MOTOR1: now also DATA_CONNECTOR1.1
- net SENSOR1 renamed FSENSOR1
- net FSENSOR1: now also DATA_CONNECTOR1.2
- net SENSOR2 renamed HSENSOR1
- net HSENSOR1: now also DATA_CONNECTOR1.15 (P15)
- net SENSOR_IN renamed SENSOR_IN_1
- net SENSOR_IN_1: now also DATA_CONNECTOR1.14 (P14)
- no-connect marks 0 -> 5
Other:
- moved on the sheet: J3

Commit message: wiring
Connections:
- net GND: no longer DATA_CONNECTOR1.13
- net GND_ESP: now also DATA_CONNECTOR1.13
Changed lines of the file:
@@
 Text Label 9000 3400 0    60   ~ 0
 MOTOR6
-$Comp
-L GND #PWR017
-U 1 1 5AC032F5
-P 9000 3800
-F 0 "#PWR017" H 9000 3550 50  0001 C CNN
-F 1 "GND" H 9000 3650 50  0000 C CNN
-F 2 "" H 9000 3800 50  0001 C CNN
-F 3 "" H 9000 3800 50  0001 C CNN
-	1    9000 3800
-	1    0    0    -1
-$EndComp
 Text Label 9000 3100 0    60   ~ 0
 SENSOR_IN_5
@@
 	10350 3700 9000 3700
 Wire Wire Line
-	10350 3800 9000 3800
+	7150 3800 10350 3800
 Connection ~ 5500 4000
 Connection ~ 5500 4100
@@
 Text Label 6500 1950 0    60   ~ 0
 +3.3V_ESP
+Wire Wire Line
+	7150 2200 7150 3800
+Connection ~ 7150 2200
 $EndSCHEMATC

Commit message: special symbols moved
Parts:
- BKOUT_L1, BKOUT_R1, ESP32_L1, ESP32_R1: symbol Conn_01x19_Female -> splitflap-rescue:Conn_01x19_Female
- C1, C3: symbol CP -> splitflap-rescue:CP
- C2: symbol C -> splitflap-rescue:C
- D1: symbol D_Bridge_+-AA-RESCUE-splitflap -> splitflap-rescue:D_Bridge_+-AA-RESCUE-splitflap
- DATA_CONNECTOR1: symbol DB25_Female -> splitflap-rescue:DB25_Female
- GND_BREAK1, VCC_BREAK1: symbol Jumper -> splitflap-rescue:Jumper
- J3: symbol Screw_Terminal_01x02 -> splitflap-rescue:Screw_Terminal_01x02
- POWER_CONNECTOR1: symbol DB9_Female -> splitflap-rescue:DB9_Female
- RV1: symbol Varistor -> splitflap-rescue:Varistor
- TRAFO1: symbol Transformer_1P_2S-RESCUE-splitflap -> splitflap-rescue:Transformer_1P_2S-RESCUE-splitflap
- TRAFO2: symbol Transformer_1P_1S-RESCUE-splitflap -> splitflap-rescue:Transformer_1P_1S-RESCUE-splitflap
- U1: symbol LD1117S33TR_SOT223 -> splitflap-rescue:LD1117S33TR_SOT223
